Commit message: Add rotational base and links to URDF model

File: test/urdf/erl1.urdf (robot description, URDF)
Before this commit: robot erl1, 3 links, 2 joints
Links:
- added link link_1, mass 5.0; collision box size=0.04 0.04 0.15; visual box size=0.04 0.04 0.15
- added link link_2, mass 5.0; collision box size=0.04 0.04 0.15; visual box size=0.04 0.04 0.15
- added link rotational_base, mass 5.0; collision cylinder length=.05 radius=.05; visual cylinder length=.05 radius=.05
Joints:
- added joint fixed_joint: type fixed, parent rotational_base, child link_1, origin xyz=0 0 0.05 rpy=0 0 0
- added joint joint_link_2: type revolute, parent link_1, child link_2, origin xyz=0 0.02 0.15 rpy=0 0 0, axis 0 1 0, limit lower=-1.57 upper=1.57 effort=2.0 velocity=2.0
- added joint joint_rotational_base: type continuous, parent link_chassis, child rotational_base, origin xyz=0 0 0.035 rpy=0 0 0, axis 0 0 1

Commit message: Added last link

File: test/urdf/erl1.urdf (robot description, URDF)
Before this commit: robot erl1, 6 links, 5 joints
Links:
- added link link_3, mass 5.0; collision box size=0.04 0.04 0.15; visual box size=0.04 0.04 0.15
Joints:
- added joint joint_link_3: type revolute, parent link_2, child link_3, origin xyz=0 0 0.15 rpy=0 0 0, axis 1 0 0, limit lower=-1.57 upper=1.57 effort=2.0 velocity=2.0
- joint joint_link_2: axis 0 1 0 -> 1 0 0; origin xyz=0 0.02 0.15 rpy=0 0 0 -> xyz=0.02 0 0.15 rpy=0 0 0

Commit message: Implemented the bridge between gazebo and ros2

File: test/urdf/erl1.urdf (robot description, URDF)
Before this commit: robot erl1, 7 links, 6 joints
Links:
- link link_chassis: mass None -> 5.0; geometry collision box size=0.5 0.3 0.07; visual box size=0.5 0.3 0.07

Commit message: Added mesh to the robot

File: test/urdf/erl1.urdf (robot description, URDF)
Before this commit: robot erl1, 7 links, 6 joints
Links:
- link link_chassis: geometry collision box size=0.5 0.25 0.07; visual mesh filename=package://test/meshes/mogi_bot.dae
Joints:
- joint joint_left_wheel: origin xyz=-0.1 0.15 0 rpy=0 0 0 -> xyz=0 0.14 0 rpy=0 0 0
- joint joint_right_wheel: origin xyz=-0.1 -0.15 0 rpy=0 0 0 -> xyz=0 -0.14 0 rpy=0 0 0
- joint joint_rotational_base: origin xyz=0 0 0.035 rpy=0 0 0 -> xyz=0 0 0.085 rpy=0 0 0

Commit message: Lidar implemented

File: test/urdf/erl1.urdf (robot description, URDF)
Before this commit: robot erl1, 7 links, 6 joints
Links:
- added link scan_link, mass 1e-5; collision box size=.1 .1 .1; visual cylinder length=0.1 radius=0.05
Joints:
- added joint scan_joint: type fixed, parent link_chassis, child scan_link, origin xyz=-0.2 0 0.19 rpy=0 0 0

Commit message: Implemented camera

File: test/urdf/erl1.urdf (robot description, URDF)
Before this commit: robot erl1, 8 links, 7 joints
Links:
- added link camera_link, mass 0.3; collision box size=0.1 0.1 0.1; visual box size=0.1 0.1 0.1
Joints:
- added joint camera_joint: type revolute, parent link_chassis, child camera_link, origin xyz=0.1 0 0.035 rpy=0 0 0, axis 0 0 1, limit lower=-1.57 upper=1.57 effort=5 velocity=1.0
